File: PhonoAmpSim.kicad_sch (KiCad schematic)
At the start: 19 parts, among them U102 ${SIM.PARAMS}, U104 ${SIM.PARAMS}

Commit message: iBom Production files Transferfunctions
Parts:
- C106: value 6n8 -> 10n
- C107: value 1n5 -> 1n
- R106: value 750k -> 1M
Changed lines of the file:
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@@
 			)
 		)
-		(property "Value" "6n8"
+		(property "Value" "10n"
 			(at 168.91 119.38 90)
 			(effects
@@
 			)
 		)
-		(property "Value" "1n5"
+		(property "Value" "1n"
 			(at 181.61 119.38 90)
 			(effects
@@
 			)
 		)
-		(property "Value" "750k"
+		(property "Value" "1M"
 			(at 168.91 102.87 90)
 			(effects
