File: PhonoAmp-rounded.kicad_pcb (KiCad board)
At the start: 2 copper layers, 72.4 x 45.7 mm, 37 parts, among them J1 Screw_Terminal_01x03, J2 Screw_Terminal_01x03, J3 Screw_Terminal_01x02, U1 NE5532, U2 TL072

Commit message: Simulation and Optimization
Parts:
- C10, C4: value 1n -> 10n
- C12, C6: value 22u -> 10u
- C3, C9: value 10n -> 47n
- R11, R4: value 1M -> 220k
- R12, R5: value 51k -> 10k
