File: PhonoAmp.kicad_sch (KiCad schematic)
At the start: 33 parts, among them J1 Screw_Terminal_01x03, J2 Screw_Terminal_01x03, J3 Screw_Terminal_01x02, U1 NE5532, U2 TL072

Commit message: Component Layout reviewed
Parts:
- added H1, H2, H3, H4: MountingHole, MountingHole:MountingHole_3mm, symbol Mechanical:MountingHole
- C1, C11, C12, C13, C14, C2, C5, C6, C7, C8: footprint Capacitor_THT:CP_Radial_D8.0mm_P2.50mm -> Capacitor_THT:CP_Radial_D8.0mm_P3.50mm
- C10, C3, C4, C9: footprint Capacitor_THT:C_Disc_D5.0mm_W2.5mm_P2.50mm -> Capacitor_THT:C_Rect_L7.2mm_W2.5mm_P5.00mm_FKS2_FKP2_MKS2_MKP2
- R1, R10, R11, R12, R13, R2, R3, R4, R5, R6, R8, R9: footprint Resistor_THT:R_Axial_DIN0411_L9.9mm_D3.6mm_P15.24mm_Horizontal -> Resistor_THT:R_Axial_DIN0207_L6.3mm_D2.5mm_P7.62mm_Horizontal

Commit message: iBom Production files Transferfunctions
Parts:
- C1, C7: footprint Capacitor_THT:CP_Radial_D8.0mm_P3.50mm -> Capacitor_THT:C_Rect_L7.2mm_W5.5mm_P5.00mm_FKS2_FKP2_MKS2_MKP2
- C10, C4: value 1n5 -> 1n
- C11, C12, C2, C5, C6, C8: footprint Capacitor_THT:CP_Radial_D8.0mm_P3.50mm -> Capacitor_THT:CP_Radial_D5.0mm_P2.00mm
- C3, C9: value 6n8 -> 10n
- R11, R4: value 750k -> 1M
Connections:
- net op1in+ renamed op1in+L
- net op1in+L: no longer C7.1, R8.1, R9.2, U1.5 (+)
- net op1in- renamed op1in-L
- net op1in-L: no longer R10.1, R13.2, U1.6 (-)
- net op2in+ renamed op2in+L
- net op2in+L: no longer R10.2, U1.7, U2.5 (+)
- net op2in- renamed op2in-L
- net op2in-L: no longer C9.2, R11.1, R14.1, U2.6 (-)
- net op2out renamed op2outL
- net op2outL: no longer C10.1, C8.2, R12.1, U2.7
- new net op1in+R: C7.1, R8.1, R9.2, U1.5 (+)
- new net op1in-R: R10.1, R13.2, U1.6 (-)
- new net op2in+R: R10.2, U1.7, U2.5 (+)
- new net op2in-R: C9.2, R11.1, R14.1, U2.6 (-)
- new net op2outR: C10.1, C8.2, R12.1, U2.7
Changed lines of the file:
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@@
 		)
 	)
-	(label "op2out"
+	(label "op2outR"
 		(at 177.8 104.14 0)
 		(fields_autoplaced yes)
@@
 		)
 	)
-	(label "op1in+"
+	(label "op1in+L"
 		(at 111.76 38.1 0)
 		(fields_autoplaced yes)
@@
 		)
 	)
-	(label "op2in-"
+	(label "op2in-L"
 		(at 152.4 43.18 0)
 		(fields_autoplaced yes)
@@
 		)
 	)
-	(label "op2out"
+	(label "op2outL"
 		(at 177.8 40.64 0)
 		(fields_autoplaced yes)
@@
 		)
 	)
-	(label "op1in-"
+	(label "op1in-L"
 		(at 119.38 43.18 0)
 		(fields_autoplaced yes)
@@
 		)
 	)
-	(label "op2in+"
+	(label "op2in+L"
 		(at 149.86 38.1 0)
 		(fields_autoplaced yes)
@@
 		)
 	)
-	(label "op2in+"
+	(label "op2in+R"
 		(at 149.86 101.6 0)
 		(fields_autoplaced yes)
@@
 		)
 	)
-	(label "op1in-"
+	(label "op1in-R"
 		(at 119.38 106.68 0)
 		(fields_autoplaced yes)
@@
 		)
 	)
-	(label "op1in+"
+	(label "op1in+R"
 		(at 111.76 101.6 0)
 		(fields_autoplaced yes)
@@
 		)
 	)
-	(label "op2in-"
+	(label "op2in-R"
 		(at 152.4 106.68 0)
 		(fields_autoplaced yes)
@@
 			)
 		)
-		(property "Footprint" "Capacitor_THT:CP_Radial_D8.0mm_P3.50mm"
+		(property "Footprint" "Capacitor_THT:CP_Radial_D5.0mm_P2.00mm"
 			(at 120.3452 134.62 0)
 			(effects
@@
 			)
 		)
-		(property "Value" "1n5"
+		(property "Value" "1n"
 			(at 181.61 129.54 90)
 			(effects
@@
 			)
 		)
-		(property "Footprint" "Capacitor_THT:CP_Radial_D8.0mm_P3.50mm"
+		(property "Footprint" "Capacitor_THT:CP_Radial_D5.0mm_P2.00mm"
 			(at 190.5 41.6052 0)
 			(effects
@@
 			)
 		)
-		(property "Value" "6n8"
+		(property "Value" "10n"
 			(at 168.91 129.54 90)
 			(effects
@@
 			)
 		)
-		(property "Footprint" "Capacitor_THT:CP_Radial_D8.0mm_P3.50mm"
+		(property "Footprint" "Capacitor_THT:CP_Radial_D5.0mm_P2.00mm"
 			(at 153.3652 71.12 0)
 			(effects
@@
 			)
 		)
-		(property "Footprint" "Capacitor_THT:CP_Radial_D8.0mm_P3.50mm"
+		(property "Footprint" "Capacitor_THT:C_Rect_L7.2mm_W5.5mm_P5.00mm_FKS2_FKP2_MKS2_MKP2"
 			(at 93.98 105.1052 0)
 			(effects
@@
 			)
 		)
-		(property "Value" "6n8"
+		(property "Value" "10n"
 			(at 168.91 66.04 90)
 			(effects
@@
 			)
 		)
-		(property "Footprint" "Capacitor_THT:CP_Radial_D8.0mm_P3.50mm"
+		(property "Footprint" "Capacitor_THT:CP_Radial_D5.0mm_P2.00mm"
 			(at 190.5 105.1052 0)
 			(effects
@@
 			)
 		)
-		(property "Footprint" "Capacitor_THT:CP_Radial_D8.0mm_P3.50mm"
+		(property "Footprint" "Capacitor_THT:C_Rect_L7.2mm_W5.5mm_P5.00mm_FKS2_FKP2_MKS2_MKP2"
 			(at 93.98 41.6052 0)
 			(effects
@@
 			)
 		)
-		(property "Value" "750k"
+		(property "Value" "1M"
 			(at 168.91 113.03 90)
 			(effects
@@
 			)
 		)
-		(property "Footprint" "Capacitor_THT:CP_Radial_D8.0mm_P3.50mm"
+		(property "Footprint" "Capacitor_THT:CP_Radial_D5.0mm_P2.00mm"
 			(at 120.3452 71.12 0)
 			(effects
@@
 			)
 		)
-		(property "Value" "1n5"
+		(property "Value" "1n"
 			(at 181.61 66.04 90)
 			(effects
@@
 			)
 		)
-		(property "Footprint" "Capacitor_THT:CP_Radial_D8.0mm_P3.50mm"
+		(property "Footprint" "Capacitor_THT:CP_Radial_D5.0mm_P2.00mm"
 			(at 153.3652 134.62 0)
 			(effects
@@
 			)
 		)
-		(property "Value" "750k"
+		(property "Value" "1M"
 			(at 168.91 49.53 90)
 			(effects

Commit message: Simulation and Optimization
Parts:
- C10, C4: value 1n -> 10n
- C12, C6: value 22u -> 10u
- C3, C9: value 10n -> 47n
- R11, R4: value 1M -> 220k
- R12, R5: value 51k -> 10k
Changed lines of the file:
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@@
 			)
 		)
-		(property "Value" "1n"
+		(property "Value" "10n"
 			(at 181.61 129.54 90)
 			(effects
@@
 			)
 		)
-		(property "Value" "51k"
+		(property "Value" "10k"
 			(at 181.61 113.03 90)
 			(effects
@@
 			)
 		)
-		(property "Value" "10n"
+		(property "Value" "47n"
 			(at 168.91 129.54 90)
 			(effects
@@
 			)
 		)
-		(property "Value" "22u"
+		(property "Value" "10u"
 			(at 156.21 67.6909 0)
 			(effects
@@
 			)
 		)
-		(property "Value" "10n"
+		(property "Value" "47n"
 			(at 168.91 66.04 90)
 			(effects
@@
 			)
 		)
-		(property "Value" "51k"
+		(property "Value" "10k"
 			(at 181.61 49.53 90)
 			(effects
@@
 			)
 		)
-		(property "Value" "1M"
+		(property "Value" "220k"
 			(at 168.91 113.03 90)
 			(effects
@@
 			)
 		)
-		(property "Value" "1n"
+		(property "Value" "10n"
 			(at 181.61 66.04 90)
 			(effects
@@
 			)
 		)
-		(property "Value" "22u"
+		(property "Value" "10u"
 			(at 156.21 131.1909 0)
 			(effects
@@
 			)
 		)
-		(property "Value" "1M"
+		(property "Value" "220k"
 			(at 168.91 49.53 90)
 			(effects
