File: PhonoAmpSim_2024-07-26.kicad_sch (KiCad schematic)
At the start: 19 parts, among them U102 ${SIM.PARAMS}, U104 ${SIM.PARAMS}

Commit message: Simulation and Optimization
Parts:
- C105: value 22u -> 10u
- C106: value 10n -> 47n
- C107: value 1n -> 10n
- R105: value 7.55k -> 1.486k
- R106: value 1M -> 220k
- R107: value 51k -> 10k
Connections:
- net op2in-: no longer C106.1, C107.2, R106.2, R107.2
- new net: C106.1, C107.2, R106.2, R107.2
Changed lines of the file:
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@@
-	)
-	(junction
-		(at 163.83 114.3)
-		(diameter 0)
-		(color 0 0 0 0)
 	)
 	(junction
@@
 	)
 	(junction
-		(at 172.72 114.3)
-		(diameter 0)
-		(color 0 0 0 0)
-	)
-	(junction
 		(at 106.68 91.44)
 		(diameter 0)
@@
 	(wire
 		(pts
-			(xy 163.83 130.81) (xy 172.72 130.81)
-		)
-		(stroke
-			(width 0)
-			(type default)
-		)
-	)
-	(wire
-		(pts
 			(xy 25.4 170.18) (xy 25.4 173.99)
 		)
@@
 	(wire
 		(pts
-			(xy 172.72 130.81) (xy 172.72 114.3)
-		)
-		(stroke
-			(width 0)
-			(type default)
-		)
-	)
-	(wire
-		(pts
 			(xy 152.4 124.46) (xy 152.4 128.27)
 		)
@@
 		(pts
 			(xy 41.91 172.72) (xy 41.91 170.18)
-		)
-		(stroke
-			(width 0)
-			(type default)
-		)
-	)
-	(wire
-		(pts
-			(xy 163.83 114.3) (xy 163.83 130.81)
 		)
 		(stroke
@@
 			)
 		)
-		(property "Value" "7.55k"
+		(property "Value" "1.486k"
 			(at 156.21 111.7599 0)
 			(effects
@@
 			)
 		)
-		(property "Value" "22u"
+		(property "Value" "10u"
 			(at 156.21 121.0309 0)
 			(effects
@@
 		(property "Description" "Polarized capacitor"
 			(at 152.4 120.65 0)
+			(effects
+				(font
+					(size 1.27 1.27)
+				)
+				(hide yes)
+			)
+		)
+		(property "Sim.Device" "C"
+			(at 0 241.3 0)
+			(effects
+				(font
+					(size 1.27 1.27)
+				)
+				(hide yes)
+			)
+		)
+		(property "Sim.Pins" "1=+ 2=-"
+			(at 0 241.3 0)
 			(effects
 				(font
@@
 			)
 		)
-		(property "Value" "10n"
+		(property "Value" "47n"
 			(at 168.91 119.38 90)
 			(effects
@@
 		(property "Description" "Unpolarized capacitor"
 			(at 168.91 114.3 0)
+			(effects
+				(font
+					(size 1.27 1.27)
+				)
+				(hide yes)
+			)
+		)
+		(property "Sim.Device" "C"
+			(at 54.61 283.21 0)
+			(effects
+				(font
+					(size 1.27 1.27)
+				)
+				(hide yes)
+			)
+		)
+		(property "Sim.Pins" "1=+ 2=-"
+			(at 54.61 283.21 0)
 			(effects
 				(font
@@
 			)
 		)
-		(property "Value" "51k"
+		(property "Value" "10k"
 			(at 181.61 102.87 90)
 			(effects
@@
 		(property "Description" "Resistor"
 			(at 181.61 106.68 0)
+			(effects
+				(font
+					(size 1.27 1.27)
+				)
+				(hide yes)
+			)
+		)
+		(property "Sim.Device" "R"
+			(at 74.93 -74.93 0)
+			(effects
+				(font
+					(size 1.27 1.27)
+				)
+				(hide yes)
+			)
+		)
+		(property "Sim.Pins" "1=+ 2=-"
+			(at 74.93 -74.93 0)
 			(effects
 				(font
@@
 			)
 		)
-		(property "Value" "1n"
+		(property "Value" "10n"
 			(at 181.61 119.38 90)
 			(effects
@@
 		(property "Description" "Unpolarized capacitor"
 			(at 181.61 114.3 0)
+			(effects
+				(font
+					(size 1.27 1.27)
+				)
+				(hide yes)
+			)
+		)
+		(property "Sim.Device" "C"
+			(at 67.31 295.91 0)
+			(effects
+				(font
+					(size 1.27 1.27)
+				)
+				(hide yes)
+			)
+		)
+		(property "Sim.Pins" "1=+ 2=-"
+			(at 67.31 295.91 0)
 			(effects
 				(font
@@
 			)
 		)
-		(property "Value" "1M"
+		(property "Value" "220k"
 			(at 168.91 102.87 90)
 			(effects
@@
 			(effects
 				(font
+					(size 1.27 1.27)
+				)
+				(hide yes)
+			)
+		)
+		(property "Sim.Device" "R"
+			(at 275.59 275.59 0)
+			(effects
+				(font
+					(size 1.27 1.27)
+				)
+				(hide yes)
+			)
+		)
+		(property "Sim.Pins" "1=+ 2=-"
+			(at 275.59 275.59 0)
+			(effects
+				(font
